File: Chess_Keypad/Chess_Keypad_for_Tandy_1650.kicad_sch (KiCad schematic)
At the start: 113 parts, among them J1 Conn_02x09_Counter_Clockwise, J2 Conn_01x08, Q1 PNP, Q2 PNP, SW1 A8, SW10 B7, SW11 C7, SW12 D7, SW13 E7, SW14 F7, SW15 G7, SW16 H7, SW17 A6, SW18 B6, SW19 C6, SW2 B8, SW20 D6, SW21 E6, SW22 F6, SW23 G6, SW24 H6, SW25 A5, SW26 B5, SW27 C5, SW28 D5, SW29 E5, SW3 C8, SW30 F5, SW31 G5, SW32 H5, SW33 A4, SW34 B4, SW35 C4, SW36 D4, SW37 E4, SW38 F4, SW39 G4, SW4 D8, SW40 H4, SW41 A3, SW42 B3, SW43 C3, SW44 D3, SW45 E3, SW46 F3, SW47 G3, SW48 H3, SW49 A2, SW5 E8, SW50 B2, SW51 C2, SW52 D2, SW53 E2, SW54 F2, SW55 G2, SW56 H2, SW57 A1, SW58 B1, SW59 C1, SW6 F8, SW60 D1, SW61 E1, SW62 F1, SW63 G1, SW64 H1, SW65 COLOUR, SW66 NEW GAME, SW67 2ndF, SW68 KING, SW69 ROOK, SW7 G8, SW70 BISHOP, SW71 TAKE BACK, SW72 LEVEL, SW73 PLAY, SW74 KNIGHT, SW75 PAWN, SW76 QUEEN, SW8 H8, SW9 A7

Commit message: Completed initial design
Parts:
- Q1, Q2: value PNP -> KSA992
Other:
- moved on the sheet: Q2, R2, R3, R6
